File: Squick/Motor_driver.sch (KiCad schematic (older format))
At the start: 9 parts, among them J7 ENK_L, J8 ENK_R, U9 TB6612FNG

Commit message: Progress with PCB and some footprint debugs
Parts:
- C16, C17, C18, C19, C20: footprint Capacitor_SMD:C_0805_2012Metric -> Capacitor_SMD:C_0603_1608Metric
Changed lines of the file:
@@
 F 0 "C19" H 4275 3450 50  0000 L CNN
 F 1 "100n" H 4225 3325 50  0000 L CNN
-F 2 "Capacitor_SMD:C_0805_2012Metric" H 4450 3375 50  0001 C CNN
+F 2 "Capacitor_SMD:C_0603_1608Metric" H 4450 3375 50  0001 C CNN
 F 3 "~" H 4450 3375 50  0001 C CNN
 	1    4450 3375
@@
 F 0 "C20" H 4525 3450 50  0000 L CNN
 F 1 "100n" H 4500 3300 50  0000 L CNN
-F 2 "Capacitor_SMD:C_0805_2012Metric" H 4700 3375 50  0001 C CNN
+F 2 "Capacitor_SMD:C_0603_1608Metric" H 4700 3375 50  0001 C CNN
 F 3 "~" H 4700 3375 50  0001 C CNN
 	1    4700 3375
@@
 F 0 "C16" H 2275 3375 50  0000 L CNN
 F 1 "100n" H 2200 3225 50  0000 L CNN
-F 2 "Capacitor_SMD:C_0805_2012Metric" H 2425 3300 50  0001 C CNN
+F 2 "Capacitor_SMD:C_0603_1608Metric" H 2425 3300 50  0001 C CNN
 F 3 "~" H 2425 3300 50  0001 C CNN
 	1    2425 3300
@@
 F 0 "C17" H 2525 3375 50  0000 L CNN
 F 1 "10u" H 2475 3225 50  0000 L CNN
-F 2 "Capacitor_SMD:C_0805_2012Metric" H 2650 3300 50  0001 C CNN
+F 2 "Capacitor_SMD:C_0603_1608Metric" H 2650 3300 50  0001 C CNN
 F 3 "~" H 2650 3300 50  0001 C CNN
 	1    2650 3300
@@
 F 0 "C18" H 2925 3325 50  0000 L CNN
 F 1 "100n" H 2875 3200 50  0000 L CNN
-F 2 "Capacitor_SMD:C_0805_2012Metric" H 2825 3300 50  0001 C CNN
+F 2 "Capacitor_SMD:C_0603_1608Metric" H 2825 3300 50  0001 C CNN
 F 3 "~" H 2825 3300 50  0001 C CNN
 	1    2825 3300

Commit message: Changed IMU and assigned 0603 footprints
Parts:
- C16, C17, C18, C19, C20: footprint Capacitor_SMD:C_0603_1608Metric -> Capacitor_SMD:C_0603_1608Metric_Pad1.05x0.95mm_HandSolder
- C21: footprint Capacitor_SMD:CP_Elec_6.3x5.9 -> Capacitor_Tantalum_SMD:CP_EIA-6032-28_Kemet-C_Pad2.25x2.35mm_HandSolder
- J7, J8: footprint Connector_PinSocket_2.54mm:PinSocket_1x06_P2.54mm_Vertical -> Connector_PinSocket_2.00mm:PinSocket_1x06_P2.00mm_Vertical
Connections:
- net L_IN1: now also U9.17 (BIN1); no longer U9.21 (AIN1)
- net L_IN2: now also U9.16 (BIN2); no longer U9.22 (AIN2)
- net M1_L: now also U9.11 (BO1), U9.12 (BO1); no longer U9.1 (AO1), U9.2 (AO1)
- net M1_R: now also U9.1 (AO1), U9.2 (AO1); no longer U9.11 (BO1), U9.12 (BO1)
- net M2_L: now also U9.7 (BO2), U9.8 (BO2); no longer U9.5 (AO2), U9.6 (AO2)
- net M2_R: now also U9.5 (AO2), U9.6 (AO2); no longer U9.7 (BO2), U9.8 (BO2)
- net PWM_L: now also U9.15 (PWMB); no longer U9.23 (PWMA)
- net PWM_R: now also U9.23 (PWMA); no longer U9.15 (PWMB)
- net R_IN1: now also U9.21 (AIN1); no longer U9.17 (BIN1)
- net R_IN2: now also U9.22 (AIN2); no longer U9.16 (BIN2)
Changed lines of the file:
@@
 EESchema Schematic File Version 4
-LIBS:Squick-cache
-EELAYER 26 0
+EELAYER 30 0
 EELAYER END
 $Descr A4 11693 8268
@@
 	1    0    0    -1
 $EndComp
+Text GLabel 3125 4100 0    50   Input ~ 0
+PWM_L
 Text GLabel 3125 4000 0    50   Input ~ 0
-PWM_L
-Text GLabel 3125 4100 0    50   Input ~ 0
 PWM_R
+Text GLabel 3125 4500 0    50   Input ~ 0
+L_IN1
+Text GLabel 3125 4600 0    50   Input ~ 0
+L_IN2
 Text GLabel 3125 4300 0    50   Input ~ 0
-L_IN1
+R_IN1
 Text GLabel 3125 4400 0    50   Input ~ 0
-L_IN2
-Text GLabel 3125 4500 0    50   Input ~ 0
-R_IN1
-Text GLabel 3125 4600 0    50   Input ~ 0
 R_IN2
 Wire Wire Line
@@
 	1    0    0    -1
 $EndComp
+Text GLabel 4325 4400 2    50   Output ~ 0
+M1_L
+Text GLabel 4325 4600 2    50   Output ~ 0
+M2_L
+Text GLabel 4325 4100 2    50   Output ~ 0
+M2_R
 Text GLabel 4325 3900 2    50   Output ~ 0
-M1_L
-Text GLabel 4325 4100 2    50   Output ~ 0
-M2_L
-Text GLabel 4325 4600 2    50   Output ~ 0
-M2_R
-Text GLabel 4325 4400 2    50   Output ~ 0
 M1_R
 Connection ~ 4025 3200
@@
 F 0 "C19" H 4275 3450 50  0000 L CNN
 F 1 "100n" H 4225 3325 50  0000 L CNN
-F 2 "Capacitor_SMD:C_0603_1608Metric" H 4450 3375 50  0001 C CNN
+F 2 "Capacitor_SMD:C_0603_1608Metric_Pad1.05x0.95mm_HandSolder" H 4450 3375 50  0001 C CNN
 F 3 "~" H 4450 3375 50  0001 C CNN
 	1    4450 3375
@@
 F 0 "C20" H 4525 3450 50  0000 L CNN
 F 1 "100n" H 4500 3300 50  0000 L CNN
-F 2 "Capacitor_SMD:C_0603_1608Metric" H 4700 3375 50  0001 C CNN
+F 2 "Capacitor_SMD:C_0603_1608Metric_Pad1.05x0.95mm_HandSolder" H 4700 3375 50  0001 C CNN
 F 3 "~" H 4700 3375 50  0001 C CNN
 	1    4700 3375
@@
 F 0 "C21" H 4991 3421 50  0000 L CNN
 F 1 "22u" H 4991 3330 50  0000 L CNN
-F 2 "Capacitor_SMD:CP_Elec_6.3x5.9" H 4900 3375 50  0001 C CNN
+F 2 "Capacitor_Tantalum_SMD:CP_EIA-6032-28_Kemet-C_Pad2.25x2.35mm_HandSolder" H 4900 3375 50  0001 C CNN
 F 3 "~" H 4900 3375 50  0001 C CNN
 	1    4900 3375
@@
 F 0 "C16" H 2275 3375 50  0000 L CNN
 F 1 "100n" H 2200 3225 50  0000 L CNN
-F 2 "Capacitor_SMD:C_0603_1608Metric" H 2425 3300 50  0001 C CNN
+F 2 "Capacitor_SMD:C_0603_1608Metric_Pad1.05x0.95mm_HandSolder" H 2425 3300 50  0001 C CNN
 F 3 "~" H 2425 3300 50  0001 C CNN
 	1    2425 3300
@@
 F 0 "C17" H 2525 3375 50  0000 L CNN
 F 1 "10u" H 2475 3225 50  0000 L CNN
-F 2 "Capacitor_SMD:C_0603_1608Metric" H 2650 3300 50  0001 C CNN
+F 2 "Capacitor_SMD:C_0603_1608Metric_Pad1.05x0.95mm_HandSolder" H 2650 3300 50  0001 C CNN
 F 3 "~" H 2650 3300 50  0001 C CNN
 	1    2650 3300
@@
 F 0 "C18" H 2925 3325 50  0000 L CNN
 F 1 "100n" H 2875 3200 50  0000 L CNN
-F 2 "Capacitor_SMD:C_0603_1608Metric" H 2825 3300 50  0001 C CNN
+F 2 "Capacitor_SMD:C_0603_1608Metric_Pad1.05x0.95mm_HandSolder" H 2825 3300 50  0001 C CNN
 F 3 "~" H 2825 3300 50  0001 C CNN
 	1    2825 3300
@@
 F 0 "J8" H 8343 3000 50  0000 C CNN
 F 1 "ENK_R" H 8343 3091 50  0000 C CNN
-F 2 "Connector_PinSocket_2.54mm:PinSocket_1x06_P2.54mm_Vertical" H 8425 3525 50  0001 C CNN
+F 2 "Connector_PinSocket_2.00mm:PinSocket_1x06_P2.00mm_Vertical" H 8425 3525 50  0001 C CNN
 F 3 "~" H 8425 3525 50  0001 C CNN
 	1    7050 3450
@@
 F 0 "J7" H 7168 3000 50  0000 C CNN
 F 1 "ENK_L" H 7168 3091 50  0000 C CNN
-F 2 "Connector_PinSocket_2.54mm:PinSocket_1x06_P2.54mm_Vertical" H 7250 3525 50  0001 C CNN
+F 2 "Connector_PinSocket_2.00mm:PinSocket_1x06_P2.00mm_Vertical" H 7250 3525 50  0001 C CNN
 F 3 "~" H 7250 3525 50  0001 C CNN
 	1    5875 3450
