File: Squick/Sensors.sch (KiCad schematic (older format))
At the start: 44 parts, among them J4 VL53L0X_L, J5 VL53L0X_F, J6 VL53L0X_R, T1 SFH-313FA, T2 SFH-313FA, T3 SFH-313FA, T4 SFH-313FA, T5 SFH-313FA, T6 SFH-313FA, U2 CD4051B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

Commit message: Created footprint for IMU
Parts:
- U8: footprint (none) -> Symbol:IMU_LSM9DS1_Adafruit4634
Changed lines of the file:
@@
 F 0 "U8" H 10175 1890 50  0000 C CNN
 F 1 "Adafruit_4634" H 10175 1799 50  0000 C CNN
-F 2 "" H 9550 2125 50  0001 C CNN
+F 2 "Symbol:IMU_LSM9DS1_Adafruit4634" H 9550 2125 50  0001 C CNN
 F 3 "" H 9550 2125 50  0001 C CNN
 	1    10100 1425

Commit message: Fixed footprints and symbol
Parts:
- U3, U5, U6, U7: footprint Varistor:transoptor_KTIR0711S -> warsztaty:KTIR0711S
Changed lines of the file:
@@
 F 0 "U7" H 8250 2050 50  0000 C CNN
 F 1 "KTIR0711S" H 8250 1959 50  0000 C CNN
-F 2 "Varistor:transoptor_KTIR0711S" H 8050 1525 50  0001 L CIN
+F 2 "warsztaty:KTIR0711S" H 8050 1525 50  0001 L CIN
 F 3 "" H 8250 1725 50  0000 L CNN
 	1    8250 1725
@@
 F 0 "U6" H 7025 2050 50  0000 C CNN
 F 1 "KTIR0711S" H 7025 1959 50  0000 C CNN
-F 2 "Varistor:transoptor_KTIR0711S" H 6825 1525 50  0001 L CIN
+F 2 "warsztaty:KTIR0711S" H 6825 1525 50  0001 L CIN
 F 3 "" H 7025 1725 50  0000 L CNN
 	1    7025 1725
@@
 F 0 "U5" H 5675 2050 50  0000 C CNN
 F 1 "KTIR0711S" H 5675 1959 50  0000 C CNN
-F 2 "Varistor:transoptor_KTIR0711S" H 5475 1525 50  0001 L CIN
+F 2 "warsztaty:KTIR0711S" H 5475 1525 50  0001 L CIN
 F 3 "" H 5675 1725 50  0000 L CNN
 	1    5675 1725
@@
 F 0 "U3" H 4300 2050 50  0000 C CNN
 F 1 "KTIR0711S" H 4300 1959 50  0000 C CNN
-F 2 "Varistor:transoptor_KTIR0711S" H 4100 1525 50  0001 L CIN
+F 2 "warsztaty:KTIR0711S" H 4100 1525 50  0001 L CIN
 F 3 "" H 4300 1725 50  0000 L CNN
 	1    4300 1725
@@
 PT_6
 $Comp
-L Squick-rescue:SFH-313FA-Squick_working T1
-U 1 1 605C6C36
-P 6475 4625
-F 0 "T1" H 6644 4496 50  0000 L CNN
-F 1 "SFH-313FA" H 6644 4405 50  0000 L CNN
-F 2 "LED_THT:LED_D5.0mm" H 6475 4375 50  0001 C CNN
-F 3 "" H 6475 4375 50  0001 C CNN
-	1    6475 4625
-	1    0    0    -1
-$EndComp
-$Comp
 L Device:R_Small R17
 U 1 1 605C83F7
@@
 Wire Wire Line
 	6600 4125 6600 4200
-Wire Wire Line
-	6600 5025 6600 5200
 $Comp
 L power:GND #PWR?
@@
 	6600 4475 6750 4475
 Connection ~ 6600 4475
-Wire Wire Line
-	6600 4475 6600 4575
 Text GLabel 6750 4475 2    50   Output ~ 0
 PT_1
@@
 Text GLabel 975  1375 2    50   Input ~ 0
 VL_XSHUT
+Wire Wire Line
+	6600 4475 6600 4575
+Wire Wire Line
+	6600 5025 6600 5200
+$Comp
+L Squick-rescue:SFH-313FA-Squick_working T1
+U 1 1 605C6C36
+P 6475 4625
+F 0 "T1" H 6644 4496 50  0000 L CNN
+F 1 "SFH-313FA" H 6644 4405 50  0000 L CNN
+F 2 "LED_THT:LED_D5.0mm" H 6475 4375 50  0001 C CNN
+F 3 "" H 6475 4375 50  0001 C CNN
+	1    6475 4625
+	1    0    0    -1
+$EndComp
 $EndSCHEMATC

Commit message: Progress with PCB and some footprint debugs
Parts:
- C14, C15: footprint Capacitor_SMD:C_0805_2012Metric -> Capacitor_SMD:C_0603_1608Metric
- U2, U4: footprint Package_DIP:DIP-16_W7.62mm_LongPads -> Package_SO:SOIC-16W_5.3x10.2mm_P1.27mm
Changed lines of the file:
@@
 F 0 "U2" H 1200 5575 50  0000 C CNN
 F 1 "CD4051B" H 1300 5500 50  0000 C CNN
-F 2 "Package_DIP:DIP-16_W7.62mm_LongPads" H 1750 3950 50  0001 L CNN
+F 2 "Package_SO:SOIC-16W_5.3x10.2mm_P1.27mm" H 1750 3950 50  0001 L CNN
 F 3 "http://www.ti.com/lit/ds/symlink/cd4052b.pdf" H 1580 4800 50  0001 C CNN
 	1    1600 4700
@@
 F 0 "C14" H 2142 3821 50  0000 L CNN
 F 1 "100n" H 2142 3730 50  0000 L CNN
-F 2 "Capacitor_SMD:C_0805_2012Metric" H 2050 3775 50  0001 C CNN
+F 2 "Capacitor_SMD:C_0603_1608Metric" H 2050 3775 50  0001 C CNN
 F 3 "~" H 2050 3775 50  0001 C CNN
 	1    2050 3775
@@
 F 0 "U4" H 4825 5625 50  0000 C CNN
 F 1 "CD4051B" H 4925 5550 50  0000 C CNN
-F 2 "Package_DIP:DIP-16_W7.62mm_LongPads" H 5375 4000 50  0001 L CNN
+F 2 "Package_SO:SOIC-16W_5.3x10.2mm_P1.27mm" H 5375 4000 50  0001 L CNN
 F 3 "http://www.ti.com/lit/ds/symlink/cd4052b.pdf" H 5205 4850 50  0001 C CNN
 	1    5225 4750
@@
 F 0 "C15" H 5767 3871 50  0000 L CNN
 F 1 "100n" H 5767 3780 50  0000 L CNN
-F 2 "Capacitor_SMD:C_0805_2012Metric" H 5675 3825 50  0001 C CNN
+F 2 "Capacitor_SMD:C_0603_1608Metric" H 5675 3825 50  0001 C CNN
 F 3 "~" H 5675 3825 50  0001 C CNN
 	1    5675 3825

Commit message: Changed IMU and assigned 0603 footprints
Parts:
- removed U8: Adafruit_4634, Symbol:IMU_LSM9DS1_Adafruit4634, symbol Squick-rescue:Adafruit_4634-Squick_working
- added U8: Adafruit_4554, symbol Squick_working:Adafruit_4554
- C14, C15: footprint Capacitor_SMD:C_0603_1608Metric -> Capacitor_SMD:C_0603_1608Metric_Pad1.05x0.95mm_HandSolder
- R10, R11, R12, R13, R14, R15, R16, R18, R19, R21, R23, R7, R8, R9: footprint Resistor_SMD:R_0805_2012Metric -> Resistor_SMD:R_0603_1608Metric_Pad1.05x0.95mm_HandSolder
- R17, R20, R22, R24, R25, R26: value 200 -> 220; footprint Resistor_SMD:R_0805_2012Metric -> Resistor_SMD:R_0603_1608Metric_Pad1.05x0.95mm_HandSolder
Connections:
- net +3.3V: now also U8.14 (Vin)
- net GND: now also U8.12 (GND), U8.4 (GND)
- net MISO: now also U8.5 (MISO)
- net MOSI: now also U8.8 (MOSI)
- net SCK: now also U8.9 (SCK)
- new net IMU_CS: U8.6 (CS)
- new net IMU_INT: U8.7 (INT)
Changed lines of the file:
@@
 EESchema Schematic File Version 4
-LIBS:Squick-cache
-EELAYER 26 0
+EELAYER 30 0
 EELAYER END
 $Descr A4 11693 8268
@@
 Text Notes 1175 850  0    100  ~ 0
 ToF Distance Sensors
-Text GLabel 10600 2175 2    50   Input ~ 0
-IMU_M
-Text GLabel 10600 2075 2    50   Input ~ 0
-IMU_AG
-Text Notes 10000 775  0    100  ~ 0
+Text Notes 9825 700  0    100  ~ 0
 IMU
-Connection ~ 9750 2125
-Wire Wire Line
-	9750 2175 9750 2125
-Wire Wire Line
-	9750 2125 9675 2125
-Wire Wire Line
-	9750 2075 9750 2125
-Text GLabel 10600 1975 2    50   Output ~ 0
+Text GLabel 10425 1825 2    50   Output ~ 0
 MOSI
-Text GLabel 9675 2125 0    50   Input ~ 0
+Text GLabel 9600 1825 0    50   Input ~ 0
 MISO
-Text GLabel 10600 1875 2    50   Output ~ 0
+Text GLabel 10425 1650 2    50   Output ~ 0
 SCK
-Text GLabel 9750 1225 0    50   Input ~ 0
-DEN
-Text GLabel 9750 1625 0    50   Output ~ 0
-IMU_DRDY
-Text GLabel 9750 1525 0    50   Output ~ 0
-IMU_INTM
-Text GLabel 9750 1325 0    50   Output ~ 0
-IMU_INT2
-Text GLabel 9750 1425 0    50   Output ~ 0
-IMU_INT1
-Text GLabel 10600 1425 2    50   BiDi ~ 0
+Text GLabel 9575 2000 0    50   Input ~ 0
+IMU_CS
+Text GLabel 10425 2000 2    50   Output ~ 0
+IMU_INT
+Text GLabel 10425 1475 2    50   BiDi ~ 0
 GND
-Text GLabel 10600 1225 2    50   Input ~ 0
+Text GLabel 10425 1125 2    50   Input ~ 0
 +3.3V
-$Comp
-L Squick-rescue:Adafruit_4634-Squick_working U?
-U 1 1 608028FE
-P 10100 1425
-AR Path="/608028FE" Ref="U?"  Part="1"
-AR Path="/607AE2DE/608028FE" Ref="U8"  Part="1"
-F 0 "U8" H 10175 1890 50  0000 C CNN
-F 1 "Adafruit_4634" H 10175 1799 50  0000 C CNN
-F 2 "Symbol:IMU_LSM9DS1_Adafruit4634" H 9550 2125 50  0001 C CNN
-F 3 "" H 9550 2125 50  0001 C CNN
-	1    10100 1425
-	1    0    0    -1
-$EndComp
 Text Notes 5700 800  0    100  ~ 0
 Line sensors
@@
 F 0 "R23" H 8550 1350 50  0000 C CNN
 F 1 "10k" H 8550 1450 50  0000 C CNN
-F 2 "Resistor_SMD:R_0805_2012Metric" V 8630 1450 50  0001 C CNN
+F 2 "Resistor_SMD:R_0603_1608Metric_Pad1.05x0.95mm_HandSolder" V 8630 1450 50  0001 C CNN
 F 3 "~" H 8700 1450 50  0001 C CNN
 	1    8700 1450
@@
 F 0 "R21" V 8043 1275 50  0000 C CNN
 F 1 "220" V 8134 1275 50  0000 C CNN
-F 2 "Resistor_SMD:R_0805_2012Metric" V 8180 1275 50  0001 C CNN
+F 2 "Resistor_SMD:R_0603_1608Metric_Pad1.05x0.95mm_HandSolder" V 8180 1275 50  0001 C CNN
 F 3 "~" H 8250 1275 50  0001 C CNN
 	1    8250 1275
@@
 F 0 "R19" H 7325 1350 50  0000 C CNN
 F 1 "10k" H 7325 1450 50  0000 C CNN
-F 2 "Resistor_SMD:R_0805_2012Metric" V 7405 1450 50  0001 C CNN
+F 2 "Resistor_SMD:R_0603_1608Metric_Pad1.05x0.95mm_HandSolder" V 7405 1450 50  0001 C CNN
 F 3 "~" H 7475 1450 50  0001 C CNN
 	1    7475 1450
@@
 F 0 "R18" V 6818 1275 50  0000 C CNN
 F 1 "220" V 6909 1275 50  0000 C CNN
-F 2 "Resistor_SMD:R_0805_2012Metric" V 6955 1275 50  0001 C CNN
+F 2 "Resistor_SMD:R_0603_1608Metric_Pad1.05x0.95mm_HandSolder" V 6955 1275 50  0001 C CNN
 F 3 "~" H 7025 1275 50  0001 C CNN
 	1    7025 1275
@@
 F 0 "R16" H 5975 1350 50  0000 C CNN
 F 1 "10k" H 5975 1450 50  0000 C CNN
-F 2 "Resistor_SMD:R_0805_2012Metric" V 6055 1450 50  0001 C CNN
+F 2 "Resistor_SMD:R_0603_1608Metric_Pad1.05x0.95mm_HandSolder" V 6055 1450 50  0001 C CNN
 F 3 "~" H 6125 1450 50  0001 C CNN
 	1    6125 1450
@@
 F 0 "R15" V 5468 1275 50  0000 C CNN
 F 1 "220" V 5559 1275 50  0000 C CNN
-F 2 "Resistor_SMD:R_0805_2012Metric" V 5605 1275 50  0001 C CNN
+F 2 "Resistor_SMD:R_0603_1608Metric_Pad1.05x0.95mm_HandSolder" V 5605 1275 50  0001 C CNN
 F 3 "~" H 5675 1275 50  0001 C CNN
 	1    5675 1275
@@
 F 0 "R14" H 4600 1350 50  0000 C CNN
 F 1 "10k" H 4600 1450 50  0000 C CNN
-F 2 "Resistor_SMD:R_0805_2012Metric" V 4680 1450 50  0001 C CNN
+F 2 "Resistor_SMD:R_0603_1608Metric_Pad1.05x0.95mm_HandSolder" V 4680 1450 50  0001 C CNN
 F 3 "~" H 4750 1450 50  0001 C CNN
 	1    4750 1450
@@
 F 0 "R13" V 4093 1275 50  0000 C CNN
 F 1 "220" V 4184 1275 50  0000 C CNN
-F 2 "Resistor_SMD:R_0805_2012Metric" V 4230 1275 50  0001 C CNN
+F 2 "Resistor_SMD:R_0603_1608Metric_Pad1.05x0.95mm_HandSolder" V 4230 1275 50  0001 C CNN
 F 3 "~" H 4300 1275 50  0001 C CNN
 	1    4300 1275
@@
 F 0 "C14" H 2142 3821 50  0000 L CNN
 F 1 "100n" H 2142 3730 50  0000 L CNN
-F 2 "Capacitor_SMD:C_0603_1608Metric" H 2050 3775 50  0001 C CNN
+F 2 "Capacitor_SMD:C_0603_1608Metric_Pad1.05x0.95mm_HandSolder" H 2050 3775 50  0001 C CNN
 F 3 "~" H 2050 3775 50  0001 C CNN
 	1    2050 3775
@@
 F 0 "R7" V 3150 4150 39  0000 C CNN
 F 1 "22" V 3225 4150 39  0000 C CNN
-F 2 "Resistor_SMD:R_0805_2012Metric" H 3275 4275 50  0001 C CNN
+F 2 "Resistor_SMD:R_0603_1608Metric_Pad1.05x0.95mm_HandSolder" H 3275 4275 50  0001 C CNN
 F 3 "~" H 3275 4275 50  0001 C CNN
 	1    3275 4275
@@
 F 0 "R8" V 3150 4350 39  0000 C CNN
 F 1 "22" V 3225 4350 39  0000 C CNN
-F 2 "Resistor_SMD:R_0805_2012Metric" H 3275 4475 50  0001 C CNN
+F 2 "Resistor_SMD:R_0603_1608Metric_Pad1.05x0.95mm_HandSolder" H 3275 4475 50  0001 C CNN
 F 3 "~" H 3275 4475 50  0001 C CNN
 	1    3275 4475
@@
 F 0 "R9" V 3150 4550 39  0000 C CNN
 F 1 "22" V 3225 4550 39  0000 C CNN
-F 2 "Resistor_SMD:R_0805_2012Metric" H 3275 4675 50  0001 C CNN
+F 2 "Resistor_SMD:R_0603_1608Metric_Pad1.05x0.95mm_HandSolder" H 3275 4675 50  0001 C CNN
 F 3 "~" H 3275 4675 50  0001 C CNN
 	1    3275 4675
@@
 F 0 "R10" V 3150 4750 39  0000 C CNN
 F 1 "22" V 3225 4750 39  0000 C CNN
-F 2 "Resistor_SMD:R_0805_2012Metric" H 3275 4875 50  0001 C CNN
+F 2 "Resistor_SMD:R_0603_1608Metric_Pad1.05x0.95mm_HandSolder" H 3275 4875 50  0001 C CNN
 F 3 "~" H 3275 4875 50  0001 C CNN
 	1    3275 4875
@@
 F 0 "R11" V 3150 4950 39  0000 C CNN
 F 1 "22" V 3225 4950 39  0000 C CNN
-F 2 "Resistor_SMD:R_0805_2012Metric" H 3275 5075 50  0001 C CNN
+F 2 "Resistor_SMD:R_0603_1608Metric_Pad1.05x0.95mm_HandSolder" H 3275 5075 50  0001 C CNN
 F 3 "~" H 3275 5075 50  0001 C CNN
 	1    3275 5075
@@
 F 0 "R12" V 3150 5150 39  0000 C CNN
 F 1 "22" V 3225 5150 39  0000 C CNN
-F 2 "Resistor_SMD:R_0805_2012Metric" H 3275 5275 50  0001 C CNN
+F 2 "Resistor_SMD:R_0603_1608Metric_Pad1.05x0.95mm_HandSolder" H 3275 5275 50  0001 C CNN
 F 3 "~" H 3275 5275 50  0001 C CNN
 	1    3275 5275
@@
 F 0 "C15" H 5767 3871 50  0000 L CNN
 F 1 "100n" H 5767 3780 50  0000 L CNN
-F 2 "Capacitor_SMD:C_0603_1608Metric" H 5675 3825 50  0001 C CNN
+F 2 "Capacitor_SMD:C_0603_1608Metric_Pad1.05x0.95mm_HandSolder" H 5675 3825 50  0001 C CNN
 F 3 "~" H 5675 3825 50  0001 C CNN
 	1    5675 3825
@@
 P 6600 4300
 F 0 "R17" H 6475 4200 39  0000 C CNN
-F 1 "200" H 6475 4300 39  0000 C CNN
-F 2 "Resistor_SMD:R_0805_2012Metric" H 6600 4300 50  0001 C CNN
+F 1 "220" H 6475 4300 39  0000 C CNN
+F 2 "Resistor_SMD:R_0603_1608Metric_Pad1.05x0.95mm_HandSolder" H 6600 4300 50  0001 C CNN
 F 3 "~" H 6600 4300 50  0001 C CNN
 	1    6600 4300
@@
 P 7475 4300
 F 0 "R20" H 7350 4200 39  0000 C CNN
-F 1 "200" H 7350 4300 39  0000 C CNN
-F 2 "Resistor_SMD:R_0805_2012Metric" H 7475 4300 50  0001 C CNN
+F 1 "220" H 7350 4300 39  0000 C CNN
+F 2 "Resistor_SMD:R_0603_1608Metric_Pad1.05x0.95mm_HandSolder" H 7475 4300 50  0001 C CNN
 F 3 "~" H 7475 4300 50  0001 C CNN
 	1    7475 4300
@@
 P 8325 4275
 F 0 "R22" H 8200 4175 39  0000 C CNN
-F 1 "200" H 8200 4275 39  0000 C CNN
-F 2 "Resistor_SMD:R_0805_2012Metric" H 8325 4275 50  0001 C CNN
+F 1 "220" H 8200 4275 39  0000 C CNN
+F 2 "Resistor_SMD:R_0603_1608Metric_Pad1.05x0.95mm_HandSolder" H 8325 4275 50  0001 C CNN
 F 3 "~" H 8325 4275 50  0001 C CNN
 	1    8325 4275
@@
 P 9125 4275
 F 0 "R24" H 9000 4175 39  0000 C CNN
-F 1 "200" H 9000 4275 39  0000 C CNN
-F 2 "Resistor_SMD:R_0805_2012Metric" H 9125 4275 50  0001 C CNN
+F 1 "220" H 9000 4275 39  0000 C CNN
+F 2 "Resistor_SMD:R_0603_1608Metric_Pad1.05x0.95mm_HandSolder" H 9125 4275 50  0001 C CNN
 F 3 "~" H 9125 4275 50  0001 C CNN
 	1    9125 4275
@@
 P 9925 4275
 F 0 "R25" H 9800 4175 39  0000 C CNN
-F 1 "200" H 9800 4275 39  0000 C CNN
-F 2 "Resistor_SMD:R_0805_2012Metric" H 9925 4275 50  0001 C CNN
+F 1 "220" H 9800 4275 39  0000 C CNN
+F 2 "Resistor_SMD:R_0603_1608Metric_Pad1.05x0.95mm_HandSolder" H 9925 4275 50  0001 C CNN
 F 3 "~" H 9925 4275 50  0001 C CNN
 	1    9925 4275
@@
 P 10725 4275
 F 0 "R26" H 10600 4175 39  0000 C CNN
-F 1 "200" H 10600 4275 39  0000 C CNN
-F 2 "Resistor_SMD:R_0805_2012Metric" H 10725 4275 50  0001 C CNN
+F 1 "220" H 10600 4275 39  0000 C CNN
+F 2 "Resistor_SMD:R_0603_1608Metric_Pad1.05x0.95mm_HandSolder" H 10725 4275 50  0001 C CNN
 F 3 "~" H 10725 4275 50  0001 C CNN
 	1    10725 4275
@@
 	1    0    0    -1
 $EndComp
+$Comp
+L Squick_working:Adafruit_4554 U8
+U 1 1 60644E3F
+P 9925 1275
+F 0 "U8" H 10000 1740 50  0000 C CNN
+F 1 "Adafruit_4554" H 10000 1649 50  0000 C CNN
+F 2 "" H 9375 1975 50  0001 C CNN
+F 3 "" H 9375 1975 50  0001 C CNN
+	1    9925 1275
+	1    0    0    -1
+$EndComp
+Text GLabel 9575 1650 0    50   BiDi ~ 0
+GND
 $EndSCHEMATC

Commit message: some debugs and small changes
Parts:
- U8: footprint (none) -> IMU_Adafruit-4554:IMU_LSM9DS1_Adafruit4634; symbol Squick_working:Adafruit_4554 -> Squick-rescue:Adafruit_4554-Squick_working
Connections:
- net +3.3V: now also U8.12 (Vin); no longer U8.14 (Vin)
- net GND: now also U8.10 (GND); no longer U8.12 (GND)
- no-connect marks 0 -> 4
Changed lines of the file:
@@
 EESchema Schematic File Version 4
-EELAYER 30 0
+LIBS:Squick-cache
+EELAYER 26 0
 EELAYER END
 $Descr A4 11693 8268
@@
 $EndComp
 $Comp
-L Squick_working:Adafruit_4554 U8
+L Squick-rescue:Adafruit_4554-Squick_working U8
 U 1 1 60644E3F
 P 9925 1275
+AR Path="/60644E3F" Ref="U8"  Part="1"
+AR Path="/607AE2DE/60644E3F" Ref="U8"  Part="1"
 F 0 "U8" H 10000 1740 50  0000 C CNN
 F 1 "Adafruit_4554" H 10000 1649 50  0000 C CNN
-F 2 "" H 9375 1975 50  0001 C CNN
+F 2 "IMU_Adafruit-4554:IMU_LSM9DS1_Adafruit4634" H 9375 1975 50  0001 C CNN
 F 3 "" H 9375 1975 50  0001 C CNN
 	1    9925 1275
@@
 Text GLabel 9575 1650 0    50   BiDi ~ 0
 GND
+NoConn ~ 9575 1475
+NoConn ~ 9575 1300
+NoConn ~ 9575 1125
+NoConn ~ 10425 1300
 $EndSCHEMATC
