File: Squick/Squick.kicad_pcb (KiCad board)
At the start: 2 copper layers, 91.5 x 92 mm, 104 parts, among them J1 BT, J10 D24V3F-5V, J2 DEBUG UART, J3 PROG, J4 VL53L0X_L, J5 VL53L0X_F, J6 VL53L0X_R, J7 ENK_L, J8 ENK_R, J9 BATT, Q1 AO3407A, Q2 AO3407A, SW1 USER_BUT_1, SW2 USER_BUT_2, SW3 RESET, SW4 ON/OFF, T1 SFH-313FA, T2 SFH-313FA, T3 SFH-313FA, T4 SFH-313FA, T5 SFH-313FA, T6 SFH-313FA, U1 STM32F411RETx, U10 LM1117-3.3, U2 CD4051B, U3 KTIR0711S, U4 CD4051B, U5 KTIR0711S, U6 KTIR0711S, U7 KTIR0711S, U8 Adafruit_4554, U9 TB6612FNG

Commit message: PCB project done!
Routing:
- net GND: track 250.6 -> 311.6 mm, vias 44 -> 55
- net PT_6: track 60.7 -> 61.4 mm
- net IR_5: track 19.5 -> 20.1 mm
- net (no net): track 0.31 -> 0.10 mm, vias 1 -> 0

Commit message: Last small debugs
Routing:
- net GND: track 311.6 -> 376.3 mm, vias 55 -> 57
- net BUT_2: track 127.6 -> 124.7 mm
- net MISO: track 102.6 -> 100.8 mm
- net LED_3: track 60.8 -> 59.9 mm
- net BT_TX: track 32.4 -> 31.6 mm
- net +3.3V: track 619.8 -> 619.0 mm
- net LED_1: track 58.4 -> 59.0 mm
- net R_IN2: track 31.9 -> 31.3 mm
- net KTIR_2: track 169.8 -> 169.9 mm, vias 12 -> 10

Commit message: Wygenerowano gerbery do produkcji płytki
Routing:
- net GND: vias 57 -> 58
Changed lines of the file:
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@@
     (thickness 1.6)
     (drawings 45)
-    (tracks 2479)
+    (tracks 2481)
     (zones 0)
     (modules 104)
@@
     (0 F.Cu signal)
     (31 B.Cu signal)
-    (32 B.Adhes user)
-    (33 F.Adhes user)
-    (34 B.Paste user)
-    (35 F.Paste user)
+    (32 B.Adhes user hide)
+    (33 F.Adhes user hide)
+    (34 B.Paste user hide)
+    (35 F.Paste user hide)
     (36 B.SilkS user)
     (37 F.SilkS user)
@@
   )
   (setup
-    (last_trace_width 0.5)
+    (last_trace_width 0.25)
     (user_trace_width 0.5)
     (user_trace_width 0.75)
@@
     (visible_elements 7FFFFFFF)
     (pcbplotparams
-      (layerselection 0x010fc_ffffffff)
+      (layerselection 0x010f0_ffffffff)
       (usegerberextensions false)
       (usegerberattributes false)
       (usegerberadvancedattributes false)
       (creategerberjobfile false)
+      (gerberprecision 5)
       (excludeedgelayer true)
       (linewidth 0.100000)
@@
       (psa4output false)
       (plotreference true)
-      (plotvalue true)
+      (plotvalue false)
       (plotinvisibletext false)
       (padsonsilk false)
@@
       (outputformat 1)
       (mirror false)
-      (drillshape 1)
+      (drillshape 0)
       (scaleselection 1)
       (outputdirectory ""))
@@
   (segment (start 204.99 123.27) (end 204.490001 123.769999) (width 0.5) (layer B.Cu) (net 2))
   (segment (start 204.490001 123.769999) (end 204.230001 123.769999) (width 0.5) (layer B.Cu) (net 2))
+  (segment (start 185.13 117.08) (end 185.13 117.08) (width 0.5) (layer F.Cu) (net 2))
+  (via (at 185.48 117) (size 0.6) (drill 0.3) (layers F.Cu B.Cu) (net 2))
   (segment (start 201.499999 107.61) (end 201.52 107.589999) (width 0.5) (layer F.Cu) (net 3))
   (segment (start 199.78 107.61) (end 201.499999 107.61) (width 0.5) (layer F.Cu) (net 3))
